Commit message: Edit controller branch

File: src/robot_pkg/urdf/Model.urdf.xacro (robot description, xacro)
@@ -1,5 +1,7 @@
-<robot name="AGV" xmlns:xacro="http://ros.org/wiki/xacro">
-  <link name="dummy_link">
-  <!-- ****************** ROBOT CONSTANTS *******************************  -->
+<?xml version="1.0"?>
+<robot name="AGV" xmlns:xacro="http://www.ros.org/wiki/xacro">
+  <!-- ######################################################################### -->
+	<!--                  ROBOT PARAMETERS        -->
+	<!-- ######################################################################### -->
   <!-- Position the wheels along the x-axis -->
   <xacro:property name="wheel_xoff" value="0.075"/>
@@ -8,5 +10,11 @@
   <!-- Position the caster wheel (collision) along the x-axis -->
   <xacro:property name="caster_collision_xoff" value="-0.075"/>
-  <!-- ****************** GROUND ***************************  -->
+  <xacro:property name="wheel_dia" value="0.15"/>
+  <xacro:property name="wheel_separate" value="0.48826"/>
+  <xacro:include filename="$(find robot_pkg)/urdf/robot_controller.xacro" />
+  <!-- ######################################################################### -->
+	<!--                 START: GROUND         -->
+	<!-- ######################################################################### -->
+  <link name="dummy_link">
   </link>
   <joint name="fixed_dummy_base" type="fixed">
@@ -15,4 +23,10 @@
     <origin xyz="0 0 0" rpy="0 0 0"/>
   </joint>
+  <!-- ######################################################################### -->
+	<!--                 END: GROUND         -->
+	<!-- ######################################################################### -->
+  <!-- ######################################################################### -->
+	<!--                 START: Base       -->
+	<!-- ######################################################################### -->
   <link name="base_link">
     <inertial>
@@ -26,7 +40,7 @@
         <mesh filename="package://robot_pkg/meshes/base_link.STL" />
       </geometry>
-      <material name="">
+      <!-- <material name="">
         <color rgba="0.894117647058823 0.913725490196078 0.929411764705882 1" />
-      </material>
+      </material> -->
     </visual>
     <collision>
@@ -37,8 +51,10 @@
     </collision>
   </link>
-  <gazebo reference="base_link">
-    <material>Gazebo/Red</material>
-  </gazebo>
-  <!-- Righ_wheel -->
+  <!-- ######################################################################### -->
+	<!--                 END: Base         -->
+	<!-- ######################################################################### -->
+ <!-- ######################################################################### -->
+ <!--                 START: Right wheel          -->
+ <!-- ######################################################################### -->
   <link name="Right_wheel">
     <inertial>
@@ -52,7 +68,7 @@
         <mesh filename="package://robot_pkg/meshes/Right_wheel.STL" />
       </geometry>
-      <material name="">
-        <color rgba="0.79216 0.81961 0.93333 1" />
-      </material>
+      <!-- <material name="">
+        <color rgba="0.79216 0.81961 0.93333 1" />
+      </material> -->
     </visual>
     <collision>
@@ -68,6 +84,13 @@
     <child link="Right_wheel" />
     <axis xyz="0 1 0" />
-  </joint>
-  <!-- Left_wheel -->
+    <limit effort="1000" velocity="1000" />
+	  <dynamics damping="1.0" friction="1.0"/>
+  </joint>
+	<!-- ######################################################################### -->
+	<!--                 END: Right wheel          -->
+	<!-- ######################################################################### -->
+	<!-- ######################################################################### -->
+	<!--                 START: Left wheel         -->
+	<!-- ######################################################################### -->
   <link name="Left_wheel">
     <inertial>
@@ -81,7 +104,7 @@
         <mesh filename="package://robot_pkg/meshes/Left_wheel.STL" />
       </geometry>
-      <material name="">
-        <color rgba="0.79216 0.81961 0.93333 1" />
-      </material>
+      <!-- <material name="">
+        <color rgba="0.79216 0.81961 0.93333 1" />
+      </material> -->
     </visual>
     <collision>
@@ -97,5 +120,13 @@
     <child link="Left_wheel" />
     <axis xyz="0 1 0" />
-  </joint>
+    <limit effort="1000" velocity="1000" />
+	  <dynamics damping="1.0" friction="1.0"/>
+  </joint>
+	<!-- ######################################################################### -->
+	<!--                 END: Caster wheel          -->
+	<!-- ######################################################################### -->
+	<!-- ######################################################################### -->
+	<!--                 START: Caster wheel          -->
+	<!-- ######################################################################### -->
   <link name="FR_Caster">
     <inertial>
@@ -126,4 +157,7 @@
     <axis xyz="0 0 0" />
   </joint>
+<!--######################################################################### -->
+<!-- ######################################################################### -->
+<!-- #########################################################################-->
   <link name="FL_Caster">
     <inertial>
@@ -154,4 +188,7 @@
     <axis xyz="0 0 0" />
   </joint>
+<!--######################################################################### -->
+<!-- ######################################################################### -->
+<!-- #########################################################################-->
   <link name="RR_Caster">
     <inertial>
@@ -182,4 +219,7 @@
     <axis xyz="0 0 0" />
   </joint>
+<!--######################################################################### -->
+<!-- ######################################################################### -->
+<!-- #########################################################################-->
   <link name="RL_Caster">
     <inertial>
@@ -210,3 +250,6 @@
     <axis xyz="0 0 0" />
   </joint>
+<!-- ######################################################################### -->
+<!--                 END: Caster wheel          -->
+<!-- ######################################################################### -->
 </robot>

File: src/robot_pkg/urdf/robot_controller.xacro (robot description, xacro)
@@ -1,3 +1,63 @@
 <?xml version="1.0"?>
-<robot>
+<robot xmlns:xacro="http://www.ros.org/wiki/xacro">
+	<gazebo reference="base_link">
+		<mu1>1</mu1>
+		<mu2>1</mu2>
+		<material>Gazebo/Blue</material>
+	</gazebo>
+	<gazebo reference="Right_wheel">
+		<mu1>1</mu1>
+		<mu2>1</mu2>
+		<material>Gazebo/Yellow</material>
+	</gazebo>
+	<gazebo reference="Left_wheel">
+		<mu1>1</mu1>
+		<mu2>1</mu2>
+		<material>Gazebo/Yellow</material>
+	</gazebo>
+	<!-- <gazebo reference="FR_Caster">
+		<mu1>0.001</mu1>
+		<mu2>0.001</mu2>
+		<material>Gazebo/Red</material>
+	</gazebo>
+	<gazebo reference="FL_Caster">
+		<mu1>0.001</mu1>
+		<mu2>0.001</mu2>
+		<material>Gazebo/Red</material>
+	</gazebo>
+	<gazebo reference="RR_Caster">
+		<mu1>0.001</mu1>
+		<mu2>0.001</mu2>
+		<material>Gazebo/Red</material>
+	</gazebo>
+	<gazebo reference="RL_Caster">
+		<mu1>0.001</mu1>
+		<mu2>0.001</mu2>
+		<material>Gazebo/Red</material>
+	</gazebo> -->
+<!-- Controller for the differential drive robot -->
+	<gazebo>
+		<plugin name='diff_drive' filename='libgazebo_ros_diff_drive.so'>
+	    		<ros>
+	        		<namespace> </namespace>
+	    		</ros>
+	    		<!-- Number of wheel pairs -->
+				<num_wheel_pairs>1</num_wheel_pairs>
+	    		<!-- wheels0-->
+	    		<left_joint>LWheel_joint</left_joint>
+	    		<right_joint>RWheel_joint</right_joint>
+	    		<!-- Kinematics -->
+	    		<wheel_separation>wheel_separate</wheel_separation>
+	    		<wheel_diameter>wheel_dia</wheel_diameter>
+	    		<!-- limits -->
+	    		<max_wheel_torque>10000</max_wheel_torque>
+	    		<max_wheel_acceleration>7.0</max_wheel_acceleration>
+	    		<!-- output -->
+	    		<publish_odom>true</publish_odom>
+	    		<publish_odom_tf>true</publish_odom_tf>
+	    		<publish_wheel_tf>true</publish_wheel_tf>
+	    		<odometry_frame>odom</odometry_frame>
+	    		<robot_base_frame>dummy_link</robot_base_frame>
+    		</plugin>
+	</gazebo>
 </robot>

Commit message: Modify urdf, launch and package

File: src/robot_pkg/urdf/Model.urdf.xacro (robot description, xacro)
@@ -31,12 +31,12 @@
   <link name="base_link">
     <inertial>
-      <origin xyz="0.0356231641912014 0.116102496743018 9.80500928933761E-08" rpy="1.5707963267949 0 0" />
+      <origin xyz="0.0356231641912014 0.116102496743018 0" rpy="1.5707963267949 0 0" />
       <mass value="14.2430877452663" />
-      <inertia ixx="0.490511050948444" ixy="-0.0515090377060454" ixz="4.23720756747739E-08" iyy="1.36650045731287" iyz="1.9746618765378E-09" izz="0.971942301144948" />
+      <inertia ixx="0.490511050948444" ixy="0" ixz="0" iyy="1.36650045731287" iyz="0" izz="0.971942301144948" />
     </inertial>
     <visual>
       <origin xyz="0 0 0.045" rpy="0 0 0" />
       <geometry>
-        <mesh filename="package://robot_pkg/meshes/base_link.STL" />
+        <mesh filename="$(find robot_pkg)/meshes/base_link.stl" />
       </geometry>
       <!-- <material name="">
@@ -47,5 +47,5 @@
       <origin xyz ="0 0 0.045" rpy = "0 0 3.141592654" />
       <geometry>
-        <mesh filename="package://robot_pkg/meshes/base_link_collision.STL" />
+        <mesh filename="$(find robot_pkg)/meshes/base_link_collision.stl" />
       </geometry>
     </collision>
@@ -61,10 +61,10 @@
       <origin xyz="0 0.0225 1.0578E-05" rpy="0 0 0" />
       <mass value="0.49011" />
-      <inertia ixx="0.00083492" ixy="1.158E-24" ixz="-1.2989E-24" iyy="0.001562" iyz="-6.0756E-20" izz="0.00083497" />
+      <inertia ixx="0.00083492" ixy="0" ixz="0" iyy="0.001562" iyz="0" izz="0.00083497" />
     </inertial>
     <visual>
       <origin xyz="0 0 0" rpy="3.141592654 0 0" />
       <geometry>
-        <mesh filename="package://robot_pkg/meshes/Right_wheel.STL" />
+        <mesh filename="$(find robot_pkg)/meshes/Right_wheel.stl" />
       </geometry>
       <!-- <material name="">
@@ -75,5 +75,5 @@
       <origin xyz="0 0 0" rpy="-1.5707963267949 0 0" />
       <geometry>
-        <mesh filename="package://robot_pkg/meshes/wheel_collision.STL" />
+        <mesh filename="$(find robot_pkg)/meshes/wheel_collision.stl" />
       </geometry>
     </collision>
@@ -97,10 +97,10 @@
       <origin xyz="-6.9389E-18 0.0225 1.0578E-05" rpy="0 0 0" />
       <mass value="0.49011" />
-      <inertia ixx="0.00083492" ixy="-1.0588E-23" ixz="-1.7579E-23" iyy="0.001562" iyz="5.7749E-20" izz="0.00083497" />
+      <inertia ixx="0.00083492" ixy="0" ixz="0" iyy="0.001562" iyz="0" izz="0.00083497" />
     </inertial>
     <visual>
       <origin xyz="0 0 0" rpy="3.141592654 0 0" />
       <geometry>
-        <mesh filename="package://robot_pkg/meshes/Left_wheel.STL" />
+        <mesh filename="$(find robot_pkg)/meshes/Left_wheel.stl" />
       </geometry>
       <!-- <material name="">
@@ -111,5 +111,5 @@
       <origin xyz="0 0 0" rpy="-1.5707963267949 0 0" />
       <geometry>
-        <mesh filename="package://robot_pkg/meshes/wheel_collision.STL" />
+        <mesh filename="$(find robot_pkg)/meshes/wheel_collision.stl" />
       </geometry>
     </collision>
@@ -133,19 +133,19 @@
       <origin xyz="-0.0033782 -0.032481 -1.3245E-09" rpy="0 0 0" />
       <mass value="0.18385" />
-      <inertia ixx="0.00019043" ixy="-1.8987E-05" ixz="1.2958E-12" iyy="0.00013092" iyz="-2.3136E-12" izz="0.00021915" />
-    </inertial>
-    <visual>
-      <origin xyz="0 0 0" rpy="1.5707963267949 0 0" />
-      <geometry>
-        <mesh filename="package://robot_pkg/meshes/FR_Caster.STL" />
-      </geometry>
-      <material name="">
-        <color rgba="0.79216 0.81961 0.93333 1" />
-      </material>
-    </visual>
-    <collision>
-      <origin xyz="0 0 ${caster_collision_xoff}" rpy="0 0 0" />
-      <geometry>
-        <mesh filename="package://robot_pkg/meshes/caster_collision.STL" />
+      <inertia ixx="0.00019043" ixy="0" ixz="0" iyy="0.00013092" iyz="0" izz="0.00021915" />
+    </inertial>
+    <visual>
+      <origin xyz="0 0 0" rpy="1.5707963267949 0 0" />
+      <geometry>
+        <mesh filename="$(find robot_pkg)/meshes/FR_Caster.stl" />
+      </geometry>
+      <material name="">
+        <color rgba="0.79216 0.81961 0.93333 1" />
+      </material>
+    </visual>
+    <collision>
+      <origin xyz="0 0 ${caster_collision_xoff}" rpy="0 0 0" />
+      <geometry>
+        <mesh filename="$(find robot_pkg)/meshes/caster_collision.stl" />
       </geometry>
     </collision>
@@ -164,19 +164,19 @@
       <origin xyz="-0.0033782 -0.032481 -1.3245E-09" rpy="1.5707963267949 0 0" />
       <mass value="0.18385" />
-      <inertia ixx="0.00019043" ixy="-1.8987E-05" ixz="1.2958E-12" iyy="0.00013092" iyz="-2.3136E-12" izz="0.00021915" />
-    </inertial>
-    <visual>
-      <origin xyz="0 0 0" rpy="1.5707963267949 0 0" />
-      <geometry>
-        <mesh filename="package://robot_pkg/meshes/FL_Caster.STL" />
-      </geometry>
-      <material name="">
-        <color rgba="0.79216 0.81961 0.93333 1" />
-      </material>
-    </visual>
-    <collision>
-      <origin xyz="0 0 ${caster_collision_xoff}" rpy="0 0 0" />
-      <geometry>
-        <mesh filename="package://robot_pkg/meshes/caster_collision.STL" />
+      <inertia ixx="0.00019043" ixy="0" ixz="0" iyy="0.00013092" iyz="0" izz="0.00021915" />
+    </inertial>
+    <visual>
+      <origin xyz="0 0 0" rpy="1.5707963267949 0 0" />
+      <geometry>
+        <mesh filename="$(find robot_pkg)/meshes/FL_Caster.stl" />
+      </geometry>
+      <material name="">
+        <color rgba="0.79216 0.81961 0.93333 1" />
+      </material>
+    </visual>
+    <collision>
+      <origin xyz="0 0 ${caster_collision_xoff}" rpy="0 0 0" />
+      <geometry>
+        <mesh filename="$(find robot_pkg)/meshes/caster_collision.stl" />
       </geometry>
     </collision>
@@ -195,19 +195,19 @@
       <origin xyz="-0.0033782 -0.032481 -1.3245E-09" rpy="0 0 0" />
       <mass value="0.18385" />
-      <inertia ixx="0.00019043" ixy="-1.8987E-05" ixz="1.2958E-12" iyy="0.00013092" iyz="-2.3136E-12" izz="0.00021915" />
-    </inertial>
-    <visual>
-      <origin xyz="0 0 0" rpy="1.5707963267949 0 0" />
-      <geometry>
-        <mesh filename="package://robot_pkg/meshes/RR_Caster.STL" />
-      </geometry>
-      <material name="">
-        <color rgba="0.79216 0.81961 0.93333 1" />
-      </material>
-    </visual>
-    <collision>
-      <origin xyz="0 0 ${caster_collision_xoff}" rpy="0 0 0" />
-      <geometry>
-        <mesh filename="package://robot_pkg/meshes/caster_collision.STL" />
+      <inertia ixx="0.00019043" ixy="0" ixz="0" iyy="0.00013092" iyz="0" izz="0.00021915" />
+    </inertial>
+    <visual>
+      <origin xyz="0 0 0" rpy="1.5707963267949 0 0" />
+      <geometry>
+        <mesh filename="$(find robot_pkg)/meshes/RR_Caster.stl" />
+      </geometry>
+      <material name="">
+        <color rgba="0.79216 0.81961 0.93333 1" />
+      </material>
+    </visual>
+    <collision>
+      <origin xyz="0 0 ${caster_collision_xoff}" rpy="0 0 0" />
+      <geometry>
+        <mesh filename="$(find robot_pkg)/meshes/caster_collision.stl" />
       </geometry>
     </collision>
@@ -226,19 +226,19 @@
       <origin xyz="-0.0033782 -0.032481 -1.3245E-09" rpy="0 0 0" />
       <mass value="0.18385" />
-      <inertia ixx="0.00019043" ixy="-1.8987E-05" ixz="1.2958E-12" iyy="0.00013092" iyz="-2.3136E-12" izz="0.00021915" />
-    </inertial>
-    <visual>
-      <origin xyz="0 0 0" rpy="1.5707963267949 0 0" />
-      <geometry>
-        <mesh filename="package://robot_pkg/meshes/RL_Caster.STL" />
-      </geometry>
-      <material name="">
-        <color rgba="0.79216 0.81961 0.93333 1" />
-      </material>
-    </visual>
-    <collision>
-      <origin xyz="0 0 ${caster_collision_xoff}" rpy="0 0 0" />
-      <geometry>
-        <mesh filename="package://robot_pkg/meshes/caster_collision.STL" />
+      <inertia ixx="0.00019043" ixy="0" ixz="0" iyy="0.00013092" iyz="0" izz="0.00021915" />
+    </inertial>
+    <visual>
+      <origin xyz="0 0 0" rpy="1.5707963267949 0 0" />
+      <geometry>
+        <mesh filename="$(find robot_pkg)/meshes/RL_Caster.stl" />
+      </geometry>
+      <material name="">
+        <color rgba="0.79216 0.81961 0.93333 1" />
+      </material>
+    </visual>
+    <collision>
+      <origin xyz="0 0 ${caster_collision_xoff}" rpy="0 0 0" />
+      <geometry>
+        <mesh filename="$(find robot_pkg)/meshes/caster_collision.stl" />
       </geometry>
     </collision>

File: src/robot_pkg/urdf/robot_controller.xacro (robot description, xacro)
@@ -7,33 +7,33 @@
 	</gazebo>
 	<gazebo reference="Right_wheel">
-		<mu1>1</mu1>
-		<mu2>1</mu2>
+		<mu1>100</mu1>
+		<mu2>100</mu2>
 		<material>Gazebo/Yellow</material>
 	</gazebo>
 	<gazebo reference="Left_wheel">
-		<mu1>1</mu1>
-		<mu2>1</mu2>
+		<mu1>100</mu1>
+		<mu2>100</mu2>
 		<material>Gazebo/Yellow</material>
 	</gazebo>
-	<!-- <gazebo reference="FR_Caster">
-		<mu1>0.001</mu1>
-		<mu2>0.001</mu2>
+	<gazebo reference="FR_Caster">
+		<mu1>0.00001</mu1>
+		<mu2>0.00001</mu2>
 		<material>Gazebo/Red</material>
 	</gazebo>
 	<gazebo reference="FL_Caster">
-		<mu1>0.001</mu1>
-		<mu2>0.001</mu2>
+		<mu1>0.00001</mu1>
+		<mu2>0.00001</mu2>
 		<material>Gazebo/Red</material>
 	</gazebo>
 	<gazebo reference="RR_Caster">
-		<mu1>0.001</mu1>
-		<mu2>0.001</mu2>
+		<mu1>0.00001</mu1>
+		<mu2>0.00001</mu2>
 		<material>Gazebo/Red</material>
 	</gazebo>
 	<gazebo reference="RL_Caster">
-		<mu1>0.001</mu1>
-		<mu2>0.001</mu2>
+		<mu1>0.00001</mu1>
+		<mu2>0.00001</mu2>
 		<material>Gazebo/Red</material>
-	</gazebo> -->
+	</gazebo>
 <!-- Controller for the differential drive robot -->
 	<gazebo>
@@ -48,9 +48,9 @@
 	    		<right_joint>RWheel_joint</right_joint>
 	    		<!-- Kinematics -->
-	    		<wheel_separation>wheel_separate</wheel_separation>
-	    		<wheel_diameter>wheel_dia</wheel_diameter>
+	    		<wheel_separation>${wheel_separate}</wheel_separation>
+	    		<wheel_diameter>${wheel_dia}</wheel_diameter>
 	    		<!-- limits -->
-	    		<max_wheel_torque>10000</max_wheel_torque>
-	    		<max_wheel_acceleration>7.0</max_wheel_acceleration>
+	    		<max_wheel_torque>20000</max_wheel_torque>
+	    		<max_wheel_acceleration>100</max_wheel_acceleration>
 	    		<!-- output -->
 	    		<publish_odom>true</publish_odom>
