Commit message: Modify rpy and xyz of links

File: src/robot_pkg/urdf/Model.urdf.xacro (robot description, xacro)
@@ -9,5 +9,5 @@
   <xacro:property name="caster_xoff" value="0.08963"/>
   <!-- Position the caster wheel (collision) along the x-axis -->
-  <xacro:property name="caster_collision_xoff" value="-0.075"/>
+  <xacro:property name="caster_collision_xoff" value="0.08963"/>
   <xacro:property name="wheel_dia" value="0.15"/>
   <xacro:property name="wheel_separate" value="0.48826"/>
@@ -45,7 +45,7 @@
     </visual>
     <collision>
-      <origin xyz ="0 0 0.045" rpy = "0 0 3.141592654" />
-      <geometry>
-        <mesh filename="$(find robot_pkg)/meshes/base_link_collision.stl" />
+      <origin xyz ="0 0 0.045" rpy = "0 0 0" />
+      <geometry>
+        <mesh filename="$(find robot_pkg)/meshes/base_link.stl" />
       </geometry>
     </collision>
@@ -73,7 +73,7 @@
     </visual>
     <collision>
-      <origin xyz="0 0 0" rpy="-1.5707963267949 0 0" />
-      <geometry>
-        <mesh filename="$(find robot_pkg)/meshes/wheel_collision.stl" />
+      <origin xyz="0 0 0" rpy="3.141592654 0 0" />
+      <geometry>
+        <mesh filename="$(find robot_pkg)/meshes/Right_wheel.stl" />
       </geometry>
     </collision>
@@ -109,7 +109,7 @@
     </visual>
     <collision>
-      <origin xyz="0 0 0" rpy="-1.5707963267949 0 0" />
-      <geometry>
-        <mesh filename="$(find robot_pkg)/meshes/wheel_collision.stl" />
+      <origin xyz="0 0 0" rpy="3.141592654 0 0" />
+      <geometry>
+        <mesh filename="$(find robot_pkg)/meshes/Left_wheel.stl" />
       </geometry>
     </collision>
@@ -145,12 +145,12 @@
     </visual>
     <collision>
-      <origin xyz="0 0 ${caster_collision_xoff}" rpy="0 0 0" />
-      <geometry>
-        <mesh filename="$(find robot_pkg)/meshes/caster_collision.stl" />
+      <origin xyz="0 0 0" rpy="1.5707963267949  0 0" />
+      <geometry>
+        <mesh filename="$(find robot_pkg)/meshes/FR_Caster.stl" />
       </geometry>
     </collision>
   </link>
   <joint name="FRC_joint" type="fixed">
-    <origin xyz="0.32 -0.1975 0.07" rpy="0 0 0" />
+    <origin xyz="0.32 -0.1975 ${caster_collision_xoff}" rpy="0 0 0" />
     <parent link="base_link" />
     <child link="FR_Caster" />
@@ -176,12 +176,12 @@
     </visual>
     <collision>
-      <origin xyz="0 0 ${caster_collision_xoff}" rpy="0 0 0" />
-      <geometry>
-        <mesh filename="$(find robot_pkg)/meshes/caster_collision.stl" />
+      <origin xyz="0 0 0" rpy="1.5707963267949 0 0" />
+      <geometry>
+        <mesh filename="$(find robot_pkg)/meshes/FL_Caster.stl" />
       </geometry>
     </collision>
   </link>
   <joint name="FLC_joint" type="fixed">
-    <origin xyz="0.32 0.1975 0.07" rpy="0 0 0" />
+    <origin xyz="0.32 0.1975 ${caster_collision_xoff}" rpy="0 0 0" />
     <parent link="base_link" />
     <child link="FL_Caster" />
@@ -207,12 +207,12 @@
     </visual>
     <collision>
-      <origin xyz="0 0 ${caster_collision_xoff}" rpy="0 0 0" />
-      <geometry>
-        <mesh filename="$(find robot_pkg)/meshes/caster_collision.stl" />
+      <origin xyz="0 0 0" rpy="1.5707963267949 0 0" />
+      <geometry>
+        <mesh filename="$(find robot_pkg)/meshes/RR_Caster.stl" />
       </geometry>
     </collision>
   </link>
   <joint name="RRC_joint" type="fixed">
-    <origin xyz="-0.32 -0.1975 0.07" rpy="0 0 0" />
+    <origin xyz="-0.32 -0.1975 ${caster_collision_xoff}" rpy="0 0 0" />
     <parent link="base_link" />
     <child link="RR_Caster" />
@@ -238,12 +238,12 @@
     </visual>
     <collision>
-      <origin xyz="0 0 ${caster_collision_xoff}" rpy="0 0 0" />
-      <geometry>
-        <mesh filename="$(find robot_pkg)/meshes/caster_collision.stl" />
+      <origin xyz="0 0 0" rpy="1.5707963267949 0 0" />
+      <geometry>
+        <mesh filename="$(find robot_pkg)/meshes/RL_Caster.stl" />
       </geometry>
     </collision>
   </link>
   <joint name="RLC_joint" type="fixed">
-    <origin xyz="-0.32 0.1975 0.07" rpy="0 0 0" />
+    <origin xyz="-0.32 0.1975 ${caster_collision_xoff}" rpy="0 0 0" />
     <parent link="base_link" />
     <child link="RL_Caster" />

File: src/robot_pkg/urdf/robot_controller.xacro (robot description, xacro)
@@ -2,36 +2,36 @@
 <robot xmlns:xacro="http://www.ros.org/wiki/xacro">
 	<gazebo reference="base_link">
-		<mu1>1</mu1>
-		<mu2>1</mu2>
+		<mu1>10</mu1>
+		<mu2>10</mu2>
 		<material>Gazebo/Blue</material>
 	</gazebo>
 	<gazebo reference="Right_wheel">
-		<mu1>100</mu1>
-		<mu2>100</mu2>
+		<mu1>10</mu1>
+		<mu2>10</mu2>
 		<material>Gazebo/Yellow</material>
 	</gazebo>
 	<gazebo reference="Left_wheel">
-		<mu1>100</mu1>
-		<mu2>100</mu2>
+		<mu1>10</mu1>
+		<mu2>10</mu2>
 		<material>Gazebo/Yellow</material>
 	</gazebo>
 	<gazebo reference="FR_Caster">
-		<mu1>0.00001</mu1>
-		<mu2>0.00001</mu2>
+		<mu1>0.1</mu1>
+		<mu2>0.1</mu2>
 		<material>Gazebo/Red</material>
 	</gazebo>
 	<gazebo reference="FL_Caster">
-		<mu1>0.00001</mu1>
-		<mu2>0.00001</mu2>
+		<mu1>0.1</mu1>
+		<mu2>0.1</mu2>
 		<material>Gazebo/Red</material>
 	</gazebo>
 	<gazebo reference="RR_Caster">
-		<mu1>0.00001</mu1>
-		<mu2>0.00001</mu2>
+		<mu1>0.1</mu1>
+		<mu2>0.1</mu2>
 		<material>Gazebo/Red</material>
 	</gazebo>
 	<gazebo reference="RL_Caster">
-		<mu1>0.00001</mu1>
-		<mu2>0.00001</mu2>
+		<mu1>0.1</mu1>
+		<mu2>0.1</mu2>
 		<material>Gazebo/Red</material>
 	</gazebo>

Commit message: Modify the dynamic and static factor

File: src/robot_pkg/urdf/Model.urdf.xacro (robot description, xacro)
@@ -5,5 +5,5 @@
 	<!-- ######################################################################### -->
   <!-- Position the wheels along the x-axis -->
-  <xacro:property name="wheel_xoff" value="0.075"/>
+  <xacro:property name="wheel_xoff" value="0.0795"/>
   <!-- Position the caster wheel (visual) along the x-axis -->
   <xacro:property name="caster_xoff" value="0.08963"/>
@@ -31,10 +31,10 @@
   <link name="base_link">
     <inertial>
-      <origin xyz="0.0356231641912014 0.116102496743018 0" rpy="1.5707963267949 0 0" />
+      <origin xyz="0 0 0.1" rpy="1.570796327 0 0" />
       <mass value="14.2430877452663" />
       <inertia ixx="0.490511050948444" ixy="0" ixz="0" iyy="1.36650045731287" iyz="0" izz="0.971942301144948" />
     </inertial>
     <visual>
-      <origin xyz="0 0 0.045" rpy="0 0 0" />
+      <origin xyz="0 0 0.03" rpy="0 0 0" />
       <geometry>
         <mesh filename="$(find robot_pkg)/meshes/base_link.stl" />
@@ -45,7 +45,7 @@
     </visual>
     <collision>
-      <origin xyz ="0 0 0.045" rpy = "0 0 0" />
-      <geometry>
-        <mesh filename="$(find robot_pkg)/meshes/base_link.stl" />
+      <origin xyz ="0 0 0.03" rpy = "0 0 3.141592654" />
+      <geometry>
+        <mesh filename="$(find robot_pkg)/meshes/base_link_collision.stl" />
       </geometry>
     </collision>
@@ -59,10 +59,10 @@
   <link name="Right_wheel">
     <inertial>
-      <origin xyz="0 0.0225 1.0578E-05" rpy="0 0 0" />
+      <origin xyz="0 0 0" rpy="-1.570796327 0 0" />
       <mass value="0.49011" />
       <inertia ixx="0.00083492" ixy="0" ixz="0" iyy="0.001562" iyz="0" izz="0.00083497" />
     </inertial>
     <visual>
-      <origin xyz="0 0 0" rpy="3.141592654 0 0" />
+      <origin xyz="0 0.0225 0" rpy="3.141592654 0 0" />
       <geometry>
         <mesh filename="$(find robot_pkg)/meshes/Right_wheel.stl" />
@@ -73,12 +73,12 @@
     </visual>
     <collision>
-      <origin xyz="0 0 0" rpy="3.141592654 0 0" />
-      <geometry>
-        <mesh filename="$(find robot_pkg)/meshes/Right_wheel.stl" />
+      <origin xyz="0 0.0225 0" rpy="-1.570796327 0 0" />
+      <geometry>
+        <mesh filename="$(find robot_pkg)/meshes/wheel_collision.stl" />
       </geometry>
     </collision>
   </link>
   <joint name="RWheel_joint" type="continuous">
-    <origin xyz="0 -0.2215 ${wheel_xoff}" rpy="0 0 0" />
+    <origin xyz="0 -0.24413 ${wheel_xoff}" rpy="0 0 0" />
     <parent link="base_link" />
     <child link="Right_wheel" />
@@ -95,10 +95,10 @@
   <link name="Left_wheel">
     <inertial>
-      <origin xyz="-6.9389E-18 0.0225 1.0578E-05" rpy="0 0 0" />
+      <origin xyz="0 0 0" rpy="-1.570796327 0 0" />
       <mass value="0.49011" />
       <inertia ixx="0.00083492" ixy="0" ixz="0" iyy="0.001562" iyz="0" izz="0.00083497" />
     </inertial>
     <visual>
-      <origin xyz="0 0 0" rpy="3.141592654 0 0" />
+      <origin xyz="0 0.0225 0" rpy="3.141592654 0 0" />
       <geometry>
         <mesh filename="$(find robot_pkg)/meshes/Left_wheel.stl" />
@@ -109,12 +109,12 @@
     </visual>
     <collision>
-      <origin xyz="0 0 0" rpy="3.141592654 0 0" />
-      <geometry>
-        <mesh filename="$(find robot_pkg)/meshes/Left_wheel.stl" />
+      <origin xyz="0 0.0225 0" rpy="-1.570796327 0 0" />
+      <geometry>
+        <mesh filename="$(find robot_pkg)/meshes/wheel_collision.stl" />
       </geometry>
     </collision>
   </link>
   <joint name="LWheel_joint" type="continuous">
-    <origin xyz="0 0.2665 ${wheel_xoff}" rpy="0 0 0" />
+    <origin xyz="0 0.24413 ${wheel_xoff}" rpy="0 0 0" />
     <parent link="base_link" />
     <child link="Left_wheel" />
@@ -131,10 +131,10 @@
   <link name="FR_Caster">
     <inertial>
-      <origin xyz="-0.0033782 -0.032481 -1.3245E-09" rpy="0 0 0" />
-      <mass value="0.18385" />
-      <inertia ixx="0.00019043" ixy="0" ixz="0" iyy="0.00013092" iyz="0" izz="0.00021915" />
-    </inertial>
-    <visual>
-      <origin xyz="0 0 0" rpy="1.5707963267949 0 0" />
+      <origin xyz="0 0 0" rpy="1.570796327 0 0" />
+      <mass value="0.18385" />
+      <inertia ixx="0.00019043" ixy="0" ixz="0" iyy="0.00013092" iyz="0" izz="0.00021915" />
+    </inertial>
+    <visual>
+      <origin xyz="0 0 0" rpy="1.570796327 0 0" />
       <geometry>
         <mesh filename="$(find robot_pkg)/meshes/FR_Caster.stl" />
@@ -145,5 +145,5 @@
     </visual>
     <collision>
-      <origin xyz="0 0 0" rpy="1.5707963267949  0 0" />
+      <origin xyz="0 0 0" rpy="1.570796327  0 0" />
       <geometry>
         <mesh filename="$(find robot_pkg)/meshes/FR_Caster.stl" />
@@ -162,10 +162,10 @@
   <link name="FL_Caster">
     <inertial>
-      <origin xyz="-0.0033782 -0.032481 -1.3245E-09" rpy="1.5707963267949 0 0" />
-      <mass value="0.18385" />
-      <inertia ixx="0.00019043" ixy="0" ixz="0" iyy="0.00013092" iyz="0" izz="0.00021915" />
-    </inertial>
-    <visual>
-      <origin xyz="0 0 0" rpy="1.5707963267949 0 0" />
+      <origin xyz="0 0 0" rpy="1.570796327 0 0" />
+      <mass value="0.18385" />
+      <inertia ixx="0.00019043" ixy="0" ixz="0" iyy="0.00013092" iyz="0" izz="0.00021915" />
+    </inertial>
+    <visual>
+      <origin xyz="0 0 0" rpy="1.570796327 0 0" />
       <geometry>
         <mesh filename="$(find robot_pkg)/meshes/FL_Caster.stl" />
@@ -176,5 +176,5 @@
     </visual>
     <collision>
-      <origin xyz="0 0 0" rpy="1.5707963267949 0 0" />
+      <origin xyz="0 0 0" rpy="1.570796327 0 0" />
       <geometry>
         <mesh filename="$(find robot_pkg)/meshes/FL_Caster.stl" />
@@ -193,10 +193,10 @@
   <link name="RR_Caster">
     <inertial>
-      <origin xyz="-0.0033782 -0.032481 -1.3245E-09" rpy="0 0 0" />
-      <mass value="0.18385" />
-      <inertia ixx="0.00019043" ixy="0" ixz="0" iyy="0.00013092" iyz="0" izz="0.00021915" />
-    </inertial>
-    <visual>
-      <origin xyz="0 0 0" rpy="1.5707963267949 0 0" />
+      <origin xyz="0 0 0" rpy="1.570796327 0 0" />
+      <mass value="0.18385" />
+      <inertia ixx="0.00019043" ixy="0" ixz="0" iyy="0.00013092" iyz="0" izz="0.00021915" />
+    </inertial>
+    <visual>
+      <origin xyz="0 0 0" rpy="1.570796327 0 0" />
       <geometry>
         <mesh filename="$(find robot_pkg)/meshes/RR_Caster.stl" />
@@ -207,5 +207,5 @@
     </visual>
     <collision>
-      <origin xyz="0 0 0" rpy="1.5707963267949 0 0" />
+      <origin xyz="0 0 0" rpy="1.570796327 0 0" />
       <geometry>
         <mesh filename="$(find robot_pkg)/meshes/RR_Caster.stl" />
@@ -229,5 +229,5 @@
     </inertial>
     <visual>
-      <origin xyz="0 0 0" rpy="1.5707963267949 0 0" />
+      <origin xyz="0 0 0" rpy="1.570796327 0 0" />
       <geometry>
         <mesh filename="$(find robot_pkg)/meshes/RL_Caster.stl" />
@@ -238,5 +238,5 @@
     </visual>
     <collision>
-      <origin xyz="0 0 0" rpy="1.5707963267949 0 0" />
+      <origin xyz="0 0 0" rpy="1.570796327 0 0" />
       <geometry>
         <mesh filename="$(find robot_pkg)/meshes/RL_Caster.stl" />

File: src/robot_pkg/urdf/robot_controller.xacro (robot description, xacro)
@@ -2,37 +2,37 @@
 <robot xmlns:xacro="http://www.ros.org/wiki/xacro">
 	<gazebo reference="base_link">
-		<mu1>10</mu1>
-		<mu2>10</mu2>
-		<material>Gazebo/Blue</material>
+		<mu1>0.5</mu1>
+		<mu2>0.3</mu2>
+		<material>Gazebo/Orange</material>
 	</gazebo>
 	<gazebo reference="Right_wheel">
-		<mu1>10</mu1>
-		<mu2>10</mu2>
-		<material>Gazebo/Yellow</material>
+		<mu1>0.5</mu1>
+		<mu2>0.3</mu2>
+		<material>Gazebo/Gray</material>
 	</gazebo>
 	<gazebo reference="Left_wheel">
-		<mu1>10</mu1>
-		<mu2>10</mu2>
-		<material>Gazebo/Yellow</material>
+		<mu1>0.5</mu1>
+		<mu2>0.3</mu2>
+		<material>Gazebo/Gray</material>
 	</gazebo>
 	<gazebo reference="FR_Caster">
-		<mu1>0.1</mu1>
-		<mu2>0.1</mu2>
-		<material>Gazebo/Red</material>
+		<mu1>0.00001</mu1>
+		<mu2>0.00001</mu2>
+		<material>Gazebo/White</material>
 	</gazebo>
 	<gazebo reference="FL_Caster">
-		<mu1>0.1</mu1>
-		<mu2>0.1</mu2>
-		<material>Gazebo/Red</material>
+		<mu1>0.00001</mu1>
+		<mu2>0.00001</mu2>
+		<material>Gazebo/White</material>
 	</gazebo>
 	<gazebo reference="RR_Caster">
-		<mu1>0.1</mu1>
-		<mu2>0.1</mu2>
-		<material>Gazebo/Red</material>
+		<mu1>0.00001</mu1>
+		<mu2>0.00001</mu2>
+		<material>Gazebo/White</material>
 	</gazebo>
 	<gazebo reference="RL_Caster">
-		<mu1>0.1</mu1>
-		<mu2>0.1</mu2>
-		<material>Gazebo/Red</material>
+		<mu1>0.00001</mu1>
+		<mu2>0.00001</mu2>
+		<material>Gazebo/White</material>
 	</gazebo>
 <!-- Controller for the differential drive robot -->
@@ -51,6 +51,6 @@
 	    		<wheel_diameter>${wheel_dia}</wheel_diameter>
 	    		<!-- limits -->
-	    		<max_wheel_torque>20000</max_wheel_torque>
-	    		<max_wheel_acceleration>100</max_wheel_acceleration>
+	    		<max_wheel_torque>5000</max_wheel_torque>
+	    		<max_wheel_acceleration>10</max_wheel_acceleration>
 	    		<!-- output -->
 	    		<publish_odom>true</publish_odom>

Commit message: Rviz run with gazebo

File: src/robot_pkg/urdf/Model.urdf.xacro (robot description, xacro)
@@ -10,7 +10,11 @@
   <!-- Position the caster wheel (collision) along the x-axis -->
   <xacro:property name="caster_collision_xoff" value="0.08963"/>
+  <!-- The parameter for wheels setup-->
   <xacro:property name="wheel_dia" value="0.15"/>
   <xacro:property name="wheel_separate" value="0.48826"/>
-  <xacro:include filename="$(find robot_pkg)/urdf/robot_controller.xacro" />
+  <!-- Include the controller plugin for gazebo-->
+  <xacro:include filename="robot_controller.xacro" />
+  <!-- Define a property for the base path to meshes -->
+  <xacro:property name="mesh_base_path" value="package://robot_pkg/"/>
   <!-- ######################################################################### -->
 	<!--                 START: GROUND         -->
@@ -38,5 +42,6 @@
       <origin xyz="0 0 0.03" rpy="0 0 0" />
       <geometry>
-        <mesh filename="$(find robot_pkg)/meshes/base_link.stl" />
+        <!-- <mesh filename="package://robot_pkg/meshes/base_link.stl" /> -->
+        <mesh filename="${mesh_base_path}/meshes/base_link.stl" />
       </geometry>
       <!-- <material name="">
@@ -47,5 +52,6 @@
       <origin xyz ="0 0 0.03" rpy = "0 0 3.141592654" />
       <geometry>
-        <mesh filename="$(find robot_pkg)/meshes/base_link_collision.stl" />
+        <!-- <mesh filename="package://robot_pkg/meshes/base_link_collision.stl" /> -->
+        <mesh filename="${mesh_base_path}/meshes/base_link_collision.stl" />
       </geometry>
     </collision>
@@ -66,5 +72,6 @@
       <origin xyz="0 0.0225 0" rpy="3.141592654 0 0" />
       <geometry>
-        <mesh filename="$(find robot_pkg)/meshes/Right_wheel.stl" />
+        <!-- <mesh filename="package://robot_pkg/meshes/Right_wheel.stl" /> -->
+        <mesh filename="${mesh_base_path}/meshes/Right_wheel.stl" />
       </geometry>
       <!-- <material name="">
@@ -75,5 +82,6 @@
       <origin xyz="0 0.0225 0" rpy="-1.570796327 0 0" />
       <geometry>
-        <mesh filename="$(find robot_pkg)/meshes/wheel_collision.stl" />
+        <!-- <mesh filename="package://robot_pkg/meshes/wheel_collision.stl" /> -->
+        <mesh filename="${mesh_base_path}/meshes/wheel_collision.stl" />
       </geometry>
     </collision>
@@ -102,5 +110,6 @@
       <origin xyz="0 0.0225 0" rpy="3.141592654 0 0" />
       <geometry>
-        <mesh filename="$(find robot_pkg)/meshes/Left_wheel.stl" />
+        <!-- <mesh filename="package://robot_pkg/meshes/Left_wheel.stl" /> -->
+        <mesh filename="${mesh_base_path}/meshes/Left_wheel.stl" />
       </geometry>
       <!-- <material name="">
@@ -111,5 +120,6 @@
       <origin xyz="0 0.0225 0" rpy="-1.570796327 0 0" />
       <geometry>
-        <mesh filename="$(find robot_pkg)/meshes/wheel_collision.stl" />
+        <!-- <mesh filename="package://robot_pkg/meshes/wheel_collision.stl" /> -->
+        <mesh filename="${mesh_base_path}/meshes/wheel_collision.stl" />
       </geometry>
     </collision>
@@ -138,5 +148,6 @@
       <origin xyz="0 0 0" rpy="1.570796327 0 0" />
       <geometry>
-        <mesh filename="$(find robot_pkg)/meshes/FR_Caster.stl" />
+        <!-- <mesh filename="package://robot_pkg/meshes/FR_Caster.stl" /> -->
+        <mesh filename="${mesh_base_path}/meshes/FR_Caster.stl" />
       </geometry>
       <material name="">
@@ -147,5 +158,6 @@
       <origin xyz="0 0 0" rpy="1.570796327  0 0" />
       <geometry>
-        <mesh filename="$(find robot_pkg)/meshes/FR_Caster.stl" />
+        <!-- <mesh filename="package://robot_pkg/meshes/FR_Caster.stl" /> -->
+        <mesh filename="${mesh_base_path}/meshes/FR_Caster.stl" />
       </geometry>
     </collision>
@@ -169,14 +181,16 @@
       <origin xyz="0 0 0" rpy="1.570796327 0 0" />
       <geometry>
-        <mesh filename="$(find robot_pkg)/meshes/FL_Caster.stl" />
-      </geometry>
-      <material name="">
-        <color rgba="0.79216 0.81961 0.93333 1" />
-      </material>
-    </visual>
-    <collision>
-      <origin xyz="0 0 0" rpy="1.570796327 0 0" />
-      <geometry>
-        <mesh filename="$(find robot_pkg)/meshes/FL_Caster.stl" />
+        <!-- <mesh filename="package://robot_pkg/meshes/FL_Caster.stl" /> -->
+        <mesh filename="${mesh_base_path}/meshes/FL_Caster.stl" />
+      </geometry>
+      <material name="">
+        <color rgba="0.79216 0.81961 0.93333 1" />
+      </material>
+    </visual>
+    <collision>
+      <origin xyz="0 0 0" rpy="1.570796327 0 0" />
+      <geometry>
+        <!-- <mesh filename="package://robot_pkg/meshes/FL_Caster.stl" /> -->
+        <mesh filename="${mesh_base_path}/meshes/FL_Caster.stl" />
       </geometry>
     </collision>
@@ -200,14 +214,16 @@
       <origin xyz="0 0 0" rpy="1.570796327 0 0" />
       <geometry>
-        <mesh filename="$(find robot_pkg)/meshes/RR_Caster.stl" />
-      </geometry>
-      <material name="">
-        <color rgba="0.79216 0.81961 0.93333 1" />
-      </material>
-    </visual>
-    <collision>
-      <origin xyz="0 0 0" rpy="1.570796327 0 0" />
-      <geometry>
-        <mesh filename="$(find robot_pkg)/meshes/RR_Caster.stl" />
+        <!-- <mesh filename="package://robot_pkg/meshes/RR_Caster.stl" /> -->
+        <mesh filename="${mesh_base_path}/meshes/RR_Caster.stl" />
+      </geometry>
+      <material name="">
+        <color rgba="0.79216 0.81961 0.93333 1" />
+      </material>
+    </visual>
+    <collision>
+      <origin xyz="0 0 0" rpy="1.570796327 0 0" />
+      <geometry>
+        <!-- <mesh filename="package://robot_pkg/meshes/RR_Caster.stl" /> -->
+        <mesh filename="${mesh_base_path}/meshes/RR_Caster.stl" />
       </geometry>
     </collision>
@@ -231,14 +247,16 @@
       <origin xyz="0 0 0" rpy="1.570796327 0 0" />
       <geometry>
-        <mesh filename="$(find robot_pkg)/meshes/RL_Caster.stl" />
-      </geometry>
-      <material name="">
-        <color rgba="0.79216 0.81961 0.93333 1" />
-      </material>
-    </visual>
-    <collision>
-      <origin xyz="0 0 0" rpy="1.570796327 0 0" />
-      <geometry>
-        <mesh filename="$(find robot_pkg)/meshes/RL_Caster.stl" />
+        <!-- <mesh filename="package://robot_pkg/meshes/RL_Caster.stl" /> -->
+        <mesh filename="${mesh_base_path}/meshes/RL_Caster.stl" />
+      </geometry>
+      <material name="">
+        <color rgba="0.79216 0.81961 0.93333 1" />
+      </material>
+    </visual>
+    <collision>
+      <origin xyz="0 0 0" rpy="1.570796327 0 0" />
+      <geometry>
+        <!-- <mesh filename="package://robot_pkg/meshes/RL_Caster.stl" /> -->
+        <mesh filename="${mesh_base_path}/meshes/RL_Caster.stl" />
       </geometry>
     </collision>

Commit message: Do nothing

File: src/robot_pkg/urdf/Model.urdf.xacro (robot description, xacro)
@@ -42,10 +42,9 @@
       <origin xyz="0 0 0.03" rpy="0 0 0" />
       <geometry>
-        <!-- <mesh filename="package://robot_pkg/meshes/base_link.stl" /> -->
         <mesh filename="${mesh_base_path}/meshes/base_link.stl" />
       </geometry>
-      <!-- <material name="">
-        <color rgba="0.894117647058823 0.913725490196078 0.929411764705882 1" />
-      </material> -->
+      <material name="orange">
+        <color rgba="1.0 0.423529411765 0.0392156862745 1.0"/>
+      </material>
     </visual>
     <collision>
@@ -75,7 +74,7 @@
         <mesh filename="${mesh_base_path}/meshes/Right_wheel.stl" />
       </geometry>
-      <!-- <material name="">
-        <color rgba="0.79216 0.81961 0.93333 1" />
-      </material> -->
+      <material name="gray">
+        <color rgba="0.5 0.5 0.5 1.0"/>
+      </material>
     </visual>
     <collision>
@@ -113,7 +112,7 @@
         <mesh filename="${mesh_base_path}/meshes/Left_wheel.stl" />
       </geometry>
-      <!-- <material name="">
-        <color rgba="0.79216 0.81961 0.93333 1" />
-      </material> -->
+      <material name="gray">
+        <color rgba="0.5 0.5 0.5 1.0"/>
+      </material>
     </visual>
     <collision>
